File: schematics/AutoFeeder_Drum-type_new/AutoFeeder_Drum-type.kicad_pcb (KiCad board)
At the start: 2 copper layers, 68.5 x 80 mm, 60 parts, among them J1 USB_C_Receptacle_6, J2 Conn_01x04, J3 Conn_01x05, J4 Conn_02x02_Odd_Even, J5 Conn_01x04, J6 Conn_02x03_Odd_Even, J7 Conn_01x04, J8 Conn_01x03, J9 Conn_01x04, M1 Motor_DC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

Commit message: Support Rev.02 PCB.
Parts:
- ?: value (none) -> Fid3
- ?: value (none) -> Fid2
- ?: renamed from REF**; value Fiducial_1mm_Mask2mm -> Fid4
- ?: value (none) -> Fid1
