File: schematics/AutoFeeder_Drum-type_2/AutoFeeder_Drum-type.kicad_sch (KiCad schematic)
At the start: 40 parts, among them J1 USB_C_Receptacle_6, J2 Conn_01x05, J3 Conn_02x02_Odd_Even, J4 Conn_02x03_Odd_Even, J5 Conn_01x01, J6 Conn_01x01, J7 Conn_01x04, M1 Motor_DC, SW1 TMHU26, U1 CNZ1023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

Commit message: Two types of sensors CNZ1023 and NJL5901 are supported. When the center button is pressed and held for 2 seconds, the hole position is memorized for one revolution, then returns to the original position. Circuit diagram is in the process of modification.
Parts:
- removed J1: USB_C_Receptacle_6, mylib:USB_C_6, symbol mylib2:USB_C_Receptacle_6
- removed R1, R2: 5.1k, Resistor_SMD:R_0603_1608Metric, symbol Device:R

Commit message: Auto Feeder 2 rev.1 ; The board is placed vertically to save space. Transmissive photo interrupter CNZ1023 can also be used.
Parts:
- removed J7: Conn_01x04, Connector_PinHeader_2.54mm:PinHeader_1x04_P2.54mm_Vertical, symbol Connector_Generic:Conn_01x04
- removed JP2: SolderJumper_3_Bridged12, Jumper:SolderJumper-3_P1.3mm_Bridged12_RoundedPad1.0x1.5mm_NumberLabels, symbol Jumper:SolderJumper_3_Bridged12
- removed RV1, RV2: 20k, Potentiometer_THT:Potentiometer_ACP_CA6-H2,5_Horizontal, symbol Device:R_Potentiometer
- removed U3: ZXBM5210-S, Package_SO:SOIC-8_3.9x4.9mm_P1.27mm, symbol Driver_Motor:ZXBM5210-S
- removed U5: NJL5901AR-1, mylib:NJL5901AR-1, symbol mylib1:CNZ1023
- added C7: 220uF, Capacitor_THT:CP_Radial_D8.0mm_P3.50mm, symbol Device:C_Polarized_Small_US
- added C8: 0.1uF, Capacitor_SMD:C_0805_2012Metric, symbol Device:C_Small
- added JP2: SolderJumper_2_Bridged, Jumper:SolderJumper-2_P1.3mm_Bridged_RoundedPad1.0x1.5mm, symbol Jumper:SolderJumper_2_Bridged
- added U2: AM2837, Package_SO:SOIC-8_3.9x4.9mm_P1.27mm, symbol mylib2:AM2837
- C3: value 10u -> 0.1uF
- C4, C5: footprint Capacitor_SMD:C_0603_1608Metric -> Capacitor_SMD:C_0805_2012Metric
Connections:
- net +5V: now also JP2.2 (B)
- net FWD: now also U2.1 (IN_A)
- net GND: now also C7.2, U2.3 (GND)
- net M1: now also M1.1 (+), C8.1, U2.7 (OUT_A), U2.8 (OUT_A); no longer M1.2 (-)
- net M2: now also M1.2 (-), C8.2, U2.5 (OUT_B), U2.6 (OUT_B); no longer M1.1 (+)
- net REV: now also U2.2 (IN_B)
- net at C3.1: now also J4.1 (Pin_1), U6.3 (IN), C7.1, JP2.1 (A), U2.4 (VCC)
Other:
- note added: "25PZF220M8X9"
- note removed: "BD6211 Max7V BD6231 Max36V"
